File: circuit/circuit.kicad_pcb (KiCad board)
At the start: 2 copper layers, 31.8 x 69.8 mm, 15 parts

Commit message: fix short
Routing:
- net GND: track 102.5 -> 97.3 mm
Changed lines of the file:
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@@
     (thickness 1.6)
     (drawings 30)
-    (tracks 110)
+    (tracks 109)
     (zones 0)
     (modules 15)
@@
   (segment (start 148.48 122.826) (end 148.48 130.37) (width 1) (layer B.Cu) (net 1))
   (segment (start 145.8976 120.2436) (end 148.48 122.826) (width 1) (layer B.Cu) (net 1))
-  (segment (start 154.94 130.37) (end 149.8 130.37) (width 1) (layer B.Cu) (net 1))
   (segment (start 135.93 120.25) (end 140.8747 120.25) (width 1) (layer B.Cu) (net 1))
   (segment (start 140.8747 120.25) (end 140.8811 120.2436) (width 1) (layer B.Cu) (net 1))
